File: schematics/microcontrollers.kicad_sch (KiCad schematic)
At the start: 2 parts, among them U4 ESP32, U5 ESP32-DevKitC

Commit message: Finished PCB Version 1
Connections:
- net Supply 3.3V renamed +3.3V
Changed lines of the file:
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@@
 		(color 0 0 0 0)
 	)
+	(junction
+		(at 101.6 81.28)
+		(diameter 0)
+		(color 0 0 0 0)
+	)
 	(no_connect
 		(at 92.71 55.88)
@@
 	(wire
 		(pts
+			(xy 101.6 78.74) (xy 101.6 81.28)
+		)
+		(stroke
+			(width 0)
+			(type default)
+		)
+	)
+	(wire
+		(pts
 			(xy 246.38 63.5) (xy 248.92 63.5)
 		)
@@
 	(wire
 		(pts
+			(xy 101.6 81.28) (xy 104.14 81.28)
+		)
+		(stroke
+			(width 0)
+			(type default)
+		)
+	)
+	(wire
+		(pts
 			(xy 246.38 78.74) (xy 248.92 78.74)
 		)
@@
 	(wire
 		(pts
-			(xy 92.71 81.28) (xy 104.14 81.28)
+			(xy 92.71 81.28) (xy 101.6 81.28)
 		)
 		(stroke
@@
 			)
 		)
+	)
+	(symbol
+		(lib_id "power:+3.3V")
+		(at 101.6 78.74 0)
+		(unit 1)
+		(exclude_from_sim no)
+		(in_bom yes)
+		(on_board yes)
+		(dnp no)
+		(fields_autoplaced yes)
+		(property "Reference" "#PWR014"
+			(at 101.6 82.55 0)
+			(effects
+				(font
+					(size 1.27 1.27)
+				)
+				(hide yes)
+			)
+		)
+		(property "Value" "+3.3V"
+			(at 101.6 73.66 0)
+			(effects
+				(font
+					(size 1.27 1.27)
+				)
+			)
+		)
+		(property "Footprint" ""
+			(at 101.6 78.74 0)
+			(effects
+				(font
+					(size 1.27 1.27)
+				)
+				(hide yes)
+			)
+		)
+		(property "Datasheet" ""
+			(at 101.6 78.74 0)
+			(effects
+				(font
+					(size 1.27 1.27)
+				)
+				(hide yes)
+			)
+		)
+		(property "Description" "Power symbol creates a global label with name \"+3.3V\""
+			(at 101.6 78.74 0)
+			(effects
+				(font
+					(size 1.27 1.27)
+				)
+				(hide yes)
+			)
+		)
+		(pin "1"
+		)
+		(instances
+			(project ""
+				(path "/bf47f329-3b1a-4bcb-94ac-b8898ea14cde/4e9b1145-8d28-4993-9235-8593e056a830"
+					(reference "#PWR014")
+					(unit 1)
+				)
+			)
+		)

Commit message: updated schematics + layout
Connections:
- net Supply 5V renamed Supply 5V ESP
Changed lines of the file:
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@@
 		)
 	)
-	(global_label "Supply 5V"
+	(global_label "Supply 5V ESP"
 		(shape input)
 		(at 41.91 81.28 180)
@@
 		)
 		(property "Intersheetrefs" "${INTERSHEET_REFS}"
-			(at 29.3698 81.28 0)
+			(at 24.7737 81.28 0)
 			(effects
 				(font
@@
 		)
 	)
-	(global_label "Supply 5V"
+	(global_label "Supply 5V ESP"
 		(shape input)
 		(at 209.55 36.83 180)
@@
 		)
 		(property "Intersheetrefs" "${INTERSHEET_REFS}"
-			(at 197.0098 36.83 0)
+			(at 192.4137 36.83 0)
 			(effects
 				(font
