File: schematics/Robofetz Mainboard.kicad_sch (KiCad schematic)
At the start: 14 parts, among them J2 PCB Power Connector, J4 Motor 1, J5 Motor 2, J6 Weapon Controller, J7 Conn_01x04_Pin, U2 DCDC, U3 ROB-14450

Commit message: updated lazout
Parts:
- H1, H2, H3, H4: footprint (none) -> MountingHole:MountingHole_2.1mm
Changed lines of the file:
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@@
 			)
 		)
-		(property "Footprint" ""
+		(property "Footprint" "MountingHole:MountingHole_2.1mm"
 			(at 60.96 162.56 0)
 			(effects
@@
 			)
 		)
-		(property "Footprint" ""
+		(property "Footprint" "MountingHole:MountingHole_2.1mm"
 			(at 35.56 162.56 0)
 			(effects
@@
 			)
 		)
-		(property "Footprint" ""
+		(property "Footprint" "MountingHole:MountingHole_2.1mm"
 			(at 34.29 149.86 0)
 			(effects
@@
 			)
 		)
-		(property "Footprint" ""
+		(property "Footprint" "MountingHole:MountingHole_2.1mm"
 			(at 59.69 149.86 0)
 			(effects
