Commit message: Apriltags working on robot

File: src/robofetz_gazebo/models/simple_diff_drive_robot/simple_diff_drive_robot.xacro (robot description, xacro)
@@ -45,4 +45,8 @@
     <!-- caster sphere -->
     <xacro:property name="I_caster" value="${(2.0/5.0)*m3*r*r}" />
+    <!-- AprilTag properties -->
+    <xacro:property name="tag_size" value="0.10" /> <!-- Size of AprilTag -->
+    <xacro:property name="tag_thickness" value="0.001" /> <!-- Thickness of tag -->
+    <xacro:property name="tag_mass" value="0.01" /> <!-- Mass of tag (10g) -->
     <!-- Complete inertia -->
     <!-- body cuboid-->
@@ -71,4 +75,17 @@
             <mass value="${m3}"/>
             <inertia ixx="${I_caster}" ixy="0.0" ixz="0.0" iyy="${I_caster}" iyz="0.0" izz="${I_caster}" />
+        </inertial>
+    </xacro:macro>
+    <!-- AprilTag inertia -->
+    <xacro:macro name="inertia_tag">
+        <inertial>
+            <origin rpy="0 0 0" xyz="0 0 0"/>
+            <mass value="${tag_mass}"/>
+            <inertia ixx="${(1.0/12.0)*tag_mass*(tag_size*tag_size + tag_thickness*tag_thickness)}"
+                     ixy="0.0"
+                     ixz="0.0"
+                     iyy="${(1.0/12.0)*tag_mass*(tag_size*tag_size + tag_thickness*tag_thickness)}"
+                     iyz="0.0"
+                     izz="${(1.0/12.0)*tag_mass*(tag_size*tag_size + tag_size*tag_size)}" />
         </inertial>
     </xacro:macro>
@@ -104,4 +121,67 @@
         <xacro:inertia_body/>
     </link>
+    <!-- AprilTag link (added on top of the robot) -->
+    <joint name="tag_joint" type="fixed">
+        <parent link="body_link"/>
+        <child link="apriltag_link"/>
+        <!-- Position the tag on top center of robot body -->
+        <!-- body height is b=0.06, tag thickness is 0.002, so place it at s1 + b/2 + tag_thickness/2 -->
+        <origin xyz="-0.03 0 ${s1 + b/2 + tag_thickness/2}" rpy="0 0 0"/>
+    </joint>
+    <link name="apriltag_link">
+        <visual>
+            <origin rpy="0 0 0" xyz="0 0 0"/>
+            <geometry>
+                <box size="${tag_size} ${tag_size} ${tag_thickness}"/>
+            </geometry>
+            <!-- Basic URDF material (fallback) -->
+            <material name="White">
+                <color rgba="1.0 1.0 1.0 1.0"/>
+            </material>
+        </visual>
+        <collision>
+            <origin rpy="0 0 0" xyz="0 0 0"/>
+            <geometry>
+                <box size="${tag_size} ${tag_size} ${tag_thickness}"/>
+            </geometry>
+        </collision>
+        <xacro:inertia_tag/>
+    </link>
+    <!-- Gazebo extension for AprilTag with PBR material (like your working SDF) -->
+    <gazebo reference="apriltag_link">
+        <!-- Physics properties -->
+        <kp>1000000.0</kp>
+        <kd>100.0</kd>
+        <mu1>0.5</mu1>
+        <mu2>0.5</mu2>
+        <!-- Material override for Gazebo -->
+        <material>Gazebo/White</material>
+        <!-- Visual override with PBR material -->
+        <visual name="apriltag_visual">
+            <geometry>
+                <box>
+                    <size>${tag_size} ${tag_size} ${tag_thickness}</size>
+                </box>
+            </geometry>
+            <material>
+                <ambient>1 1 1 1</ambient>
+                <diffuse>1 1 1 1</diffuse>
+                <specular>0.5 0.5 0.5 1</specular>
+                <pbr>
+                    <metal>
+                        <!-- Use the texture path that works in your SDF -->
+                        <!-- Option 1: Relative path (like your SDF) -->
+                        <albedo_map>file://$(find robofetz_gazebo)/models/simple_diff_drive_robot/top_apriltag.png</albedo_map>
+                        <!-- Option 2: Using find command -->
+                        <!-- <albedo_map>$(find robofetz_gazebo)/models/simple_diff_drive_robot/apriltag.png</albedo_map> -->
+                        <!-- Option 3: Absolute path to your texture -->
+                        <!-- <albedo_map>/home/$(env USER)/catkin_ws/src/robofetz_gazebo/models/simple_diff_drive_robot/apriltag.png</albedo_map> -->
+                        <roughness>0.5</roughness>
+                        <metalness>0.0</metalness>
+                    </metal>
+                </pbr>
+            </material>
+        </visual>
+    </gazebo>
     <!-- Wheel1 of the robot -->
     <joint name="wheel1_joint" type="continuous" >

Commit message: added correct apriltags

File: src/robofetz_gazebo/models/simple_diff_drive_robot/simple_diff_drive_robot.xacro (robot description, xacro)
@@ -121,13 +121,12 @@
         <xacro:inertia_body/>
     </link>
-    <!-- AprilTag link (added on top of the robot) -->
-    <joint name="tag_joint" type="fixed">
-        <parent link="body_link"/>
-        <child link="apriltag_link"/>
-        <!-- Position the tag on top center of robot body -->
-        <!-- body height is b=0.06, tag thickness is 0.002, so place it at s1 + b/2 + tag_thickness/2 -->
+    <!-- Top AprilTag link (added on top of the robot) -->
+    <joint name="top_tag_joint" type="fixed">
+        <parent link="body_link"/>
+        <child link="top_apriltag_link"/>
+        <!-- Position the tag on top center of robot body, slightly offset to front -->
         <origin xyz="-0.03 0 ${s1 + b/2 + tag_thickness/2}" rpy="0 0 0"/>
     </joint>
-    <link name="apriltag_link">
+    <link name="top_apriltag_link">
         <visual>
             <origin rpy="0 0 0" xyz="0 0 0"/>
@@ -148,6 +147,34 @@
         <xacro:inertia_tag/>
     </link>
-    <!-- Gazebo extension for AprilTag with PBR material (like your working SDF) -->
-    <gazebo reference="apriltag_link">
+    <!-- Bottom AprilTag link (added on bottom of the robot) -->
+    <joint name="bottom_tag_joint" type="fixed">
+        <parent link="body_link"/>
+        <child link="bottom_apriltag_link"/>
+        <!-- Position the tag on bottom center of robot body -->
+        <!-- Rotation 180 degrees around X axis to face downward -->
+        <!-- Position: s1 - b/2 - tag_thickness/2 (below the body) -->
+        <origin xyz="-0.03 0 ${s1 - b/2 - tag_thickness/2}" rpy="${pi_const} 0 0"/>
+    </joint>
+    <link name="bottom_apriltag_link">
+        <visual>
+            <origin rpy="0 0 0" xyz="0 0 0"/>
+            <geometry>
+                <box size="${tag_size} ${tag_size} ${tag_thickness}"/>
+            </geometry>
+            <!-- Basic URDF material (fallback) -->
+            <material name="White">
+                <color rgba="1.0 1.0 1.0 1.0"/>
+            </material>
+        </visual>
+        <collision>
+            <origin rpy="0 0 0" xyz="0 0 0"/>
+            <geometry>
+                <box size="${tag_size} ${tag_size} ${tag_thickness}"/>
+            </geometry>
+        </collision>
+        <xacro:inertia_tag/>
+    </link>
+    <!-- Gazebo extension for Top AprilTag with PBR material -->
+    <gazebo reference="top_apriltag_link">
         <!-- Physics properties -->
         <kp>1000000.0</kp>
@@ -158,5 +185,5 @@
         <material>Gazebo/White</material>
         <!-- Visual override with PBR material -->
-        <visual name="apriltag_visual">
+        <visual name="top_apriltag_visual">
             <geometry>
                 <box>
@@ -170,11 +197,5 @@
                 <pbr>
                     <metal>
-                        <!-- Use the texture path that works in your SDF -->
-                        <!-- Option 1: Relative path (like your SDF) -->
                         <albedo_map>file://$(find robofetz_gazebo)/models/simple_diff_drive_robot/top_apriltag.png</albedo_map>
-                        <!-- Option 2: Using find command -->
-                        <!-- <albedo_map>$(find robofetz_gazebo)/models/simple_diff_drive_robot/apriltag.png</albedo_map> -->
-                        <!-- Option 3: Absolute path to your texture -->
-                        <!-- <albedo_map>/home/$(env USER)/catkin_ws/src/robofetz_gazebo/models/simple_diff_drive_robot/apriltag.png</albedo_map> -->
                         <roughness>0.5</roughness>
                         <metalness>0.0</metalness>
@@ -184,4 +205,35 @@
         </visual>
     </gazebo>
+    <!-- Gazebo extension for Bottom AprilTag with PBR material -->
+    <gazebo reference="bottom_apriltag_link">
+        <!-- Physics properties -->
+        <kp>1000000.0</kp>
+        <kd>100.0</kd>
+        <mu1>0.5</mu1>
+        <mu2>0.5</mu2>
+        <!-- Material override for Gazebo -->
+        <material>Gazebo/White</material>
+        <!-- Visual override with PBR material -->
+        <visual name="bottom_apriltag_visual">
+            <geometry>
+                <box>
+                    <size>${tag_size} ${tag_size} ${tag_thickness}</size>
+                </box>
+            </geometry>
+            <material>
+                <ambient>1 1 1 1</ambient>
+                <diffuse>1 1 1 1</diffuse>
+                <specular>0.5 0.5 0.5 1</specular>
+                <pbr>
+                    <metal>
+                        <!-- Use a different texture for bottom tag if desired -->
+                        <albedo_map>file://$(find robofetz_gazebo)/models/simple_diff_drive_robot/bottom_apriltag.png</albedo_map>
+                        <roughness>0.5</roughness>
+                        <metalness>0.0</metalness>
+                    </metal>
+                </pbr>
+            </material>
+        </visual>
+    </gazebo>
     <!-- Wheel1 of the robot -->
     <joint name="wheel1_joint" type="continuous" >

Commit message: some good progress on urdf

File: src/robofetz_gazebo/models/simple_diff_drive_robot/simple_diff_drive_robot.xacro (robot description, xacro)
@@ -8,15 +8,23 @@
     <xacro:property name="pi_const" value="3.14159265" />
     <!-- Body Dimensions -->
-    <xacro:property name="a" value="0.18" />
-    <xacro:property name="b" value="0.06" />
-    <xacro:property name="c" value="0.13" />
+    <!-- Length -->
+    <xacro:property name="a" value="0.140" />
+    <!-- Height -->
+    <xacro:property name="b" value="0.054" />
+    <!-- Width -->
+    <xacro:property name="c" value="0.14" />
     <!-- Wheel and caster radius -->
-    <xacro:property name="r" value="0.04" />
+    <xacro:property name="r" value="0.034" />
     <!-- Wheel width -->
-    <xacro:property name="d" value="0.01" />
+    <xacro:property name="d" value="0.026" />
+    <!-- Wheel Offset to chassis in Y axis -->
+    <xacro:property name="e" value="0.00675" />
     <xacro:property name="s1" value="${r}" />
-    <xacro:property name="s2" value="${a/2.0-r/2.0}" />
-    <xacro:property name="s3" value="${a/2.0-r}" />
-    <xacro:property name="s4" value="${c/2.0+d/2.0}" />
+    <!-- Wheel Position relative to body center X axis -->
+    <xacro:property name="s2" value="${a/2.0-0.04075}" />
+    <!-- Caster Offset -->
+    <xacro:property name="s3" value="${a+r}" />
+    <!-- Wheel position relative to body center Y axis -->
+    <xacro:property name="s4" value="${c/2.0+d/2+e}" />
     <!-- ########################## -->
     <!--      Mass and inertia      -->
@@ -47,5 +55,5 @@
     <xacro:property name="I_caster" value="${(2.0/5.0)*m3*r*r}" />
     <!-- AprilTag properties -->
-    <xacro:property name="tag_size" value="0.10" /> <!-- Size of AprilTag -->
+    <xacro:property name="tag_size" value="0.14" /> <!-- Size of AprilTag -->
     <xacro:property name="tag_thickness" value="0.001" /> <!-- Thickness of tag -->
     <xacro:property name="tag_mass" value="0.01" /> <!-- Mass of tag (10g) -->
@@ -127,5 +135,5 @@
         <child link="$(arg prefix)top_apriltag_link"/>
         <!-- Position the tag on top center of robot body, slightly offset to front -->
-        <origin xyz="-0.03 0 ${s1 + b/2 + tag_thickness/2}" rpy="0 0 0"/>
+        <origin xyz="0 0 ${s1 + b/2 + tag_thickness/2}" rpy="0 0 0"/>
     </joint>
     <link name="$(arg prefix)top_apriltag_link">
@@ -155,5 +163,5 @@
         <!-- Rotation 180 degrees around X axis to face downward -->
         <!-- Position: s1 - b/2 - tag_thickness/2 (below the body) -->
-        <origin xyz="-0.03 0 ${s1 - b/2 - tag_thickness/2}" rpy="${pi_const} 0 0"/>
+        <origin xyz="0 0 ${s1 - b/2 - tag_thickness/2}" rpy="${pi_const} 0 0"/>
     </joint>
     <link name="$(arg prefix)bottom_apriltag_link">
