Commit message: robot adjusted to testbot

File: src/robofetz_gazebo/models/simple_diff_drive_robot/simple_diff_drive_robot.xacro (robot description, xacro)
@@ -8,9 +8,6 @@
     <xacro:property name="pi_const" value="3.14159265" />
     <!-- Body Dimensions -->
-    <!-- Length -->
     <xacro:property name="a" value="0.140" />
-    <!-- Height -->
     <xacro:property name="b" value="0.054" />
-    <!-- Width -->
     <xacro:property name="c" value="0.14" />
     <!-- Wheel and caster radius -->
@@ -21,46 +18,40 @@
     <xacro:property name="e" value="0.00675" />
     <xacro:property name="s1" value="${r}" />
-    <!-- Wheel Position relative to body center X axis -->
     <xacro:property name="s2" value="${a/2.0-0.04075}" />
-    <!-- Caster Offset -->
     <xacro:property name="s3" value="${a+r}" />
-    <!-- Wheel position relative to body center Y axis -->
     <xacro:property name="s4" value="${c/2.0+d/2+e}" />
+    <!-- Upright support box dimensions (replacing cylinder) -->
+    <xacro:property name="f" value="0.0049"/>
+    <xacro:property name="support_width" value="${2*f}" />
+    <xacro:property name="support_height" value="${2*r-2*f}" />
     <!-- ########################## -->
     <!--      Mass and inertia      -->
     <!-- ########################## -->
     <!-- Material Density -->
-    <!-- body -->
     <xacro:property name="d1" value="1430.0" />
-    <!-- wheel -->
     <xacro:property name="d2" value="1430.0" />
-    <!-- caster -->
     <xacro:property name="d3" value="1430.0" />
     <!-- Mass -->
-    <!-- body cuboid-->
     <xacro:property name="m1" value="${d1*a*b*c}" />
-    <!-- wheel cylinder-->
     <xacro:property name="m2" value="${d2*pi_const*r*r*d}" />
-    <!-- caster sphere -->
-    <xacro:property name="m3" value="${d3*(4.0/3.0)*pi_const*r*r*r}" />
+    <!-- Updated mass calculation for box support -->
+    <xacro:property name="m3" value="${d3*support_width*support_width*support_height}" />
     <!-- Inertia -->
-    <!-- body cuboid-->
     <xacro:property name="Ix_body" value="${(1.0/12.0)*m1*(b*b+c*c)}" />
     <xacro:property name="Iy_body" value="${(1.0/12.0)*m1*(a*a+b*b)}" />
     <xacro:property name="Iz_body" value="${(1.0/12.0)*m1*(a*a+c*c)}" />
-    <!-- wheel cylinder-->
     <xacro:property name="Iz_wheel" value="${0.5*m2*r*r}" />
     <xacro:property name="I_wheel" value="${(1.0/12.0)*m2*(3.0*r*r+d*d)}" />
-    <!-- caster sphere -->
-    <xacro:property name="I_caster" value="${(2.0/5.0)*m3*r*r}" />
+    <!-- Updated inertia for box support -->
+    <xacro:property name="I_support_x" value="${(1.0/12.0)*m3*(support_width*support_width + support_height*support_height)}" />
+    <xacro:property name="I_support_y" value="${(1.0/12.0)*m3*(support_width*support_width + support_height*support_height)}" />
+    <xacro:property name="I_support_z" value="${(1.0/12.0)*m3*(support_width*support_width + support_width*support_width)}" />
     <!-- AprilTag properties -->
-    <xacro:property name="tag_size" value="0.14" /> <!-- Size of AprilTag -->
-    <xacro:property name="tag_thickness" value="0.001" /> <!-- Thickness of tag -->
-    <xacro:property name="tag_mass" value="0.01" /> <!-- Mass of tag (10g) -->
-    <!-- Complete inertia -->
-    <!-- body cuboid-->
+    <xacro:property name="tag_size" value="0.14" />
+    <xacro:property name="tag_thickness" value="0.001" />
+    <xacro:property name="tag_mass" value="0.01" />
+    <!-- Complete inertia macros -->
     <xacro:macro name="inertia_body">
         <inertial>
-            <!-- Displacement and orientation of the center of the mass frame of the link with respect to parent coordinate system -->
             <origin rpy="0 0 0" xyz="0 0 ${s1}"/>
             <mass value="${m1}"/>
@@ -68,23 +59,18 @@
         </inertial>
     </xacro:macro>
-    <!-- wheel cylinder-->
     <xacro:macro name="inertia_wheel">
         <inertial>
-            <!-- Displacement and orientation of the center of the mass frame of the link with respect to parent coordinate system -->
-            <origin rpy="${pi_const/2.0} 0 0" xyz="0 0 0"/> <!-- rpy in radiants -->
+            <origin rpy="${pi_const/2.0} 0 0" xyz="0 0 0"/>
             <mass value="${m2}"/>
             <inertia ixx="${I_wheel}" ixy="0.0" ixz="0.0" iyy="${I_wheel}" iyz="0.0" izz="${Iz_wheel}" />
         </inertial>
     </xacro:macro>
-    <!-- caster sphere -->
-    <xacro:macro name="inertia_caster">
-        <inertial>
-            <!-- Displacement and orientation of the center of the mass frame of the link with respect to parent coordinate system -->
-            <origin rpy="0 0 0" xyz="0 0 0"/> <!-- rpy in radiants -->
+    <xacro:macro name="inertia_support">
+        <inertial>
+            <origin rpy="0 0 0" xyz="0 0 0"/>
             <mass value="${m3}"/>
-            <inertia ixx="${I_caster}" ixy="0.0" ixz="0.0" iyy="${I_caster}" iyz="0.0" izz="${I_caster}" />
-        </inertial>
-    </xacro:macro>
-    <!-- AprilTag inertia -->
+            <inertia ixx="${I_support_x}" ixy="0.0" ixz="0.0" iyy="${I_support_y}" iyz="0.0" izz="${I_support_z}" />
+        </inertial>
+    </xacro:macro>
     <xacro:macro name="inertia_tag">
         <inertial>
@@ -92,6 +78,5 @@
             <mass value="${tag_mass}"/>
             <inertia ixx="${(1.0/12.0)*tag_mass*(tag_size*tag_size + tag_thickness*tag_thickness)}"
-                     ixy="0.0"
-                     ixz="0.0"
+                     ixy="0.0" ixz="0.0"
                      iyy="${(1.0/12.0)*tag_mass*(tag_size*tag_size + tag_thickness*tag_thickness)}"
                      iyz="0.0"
@@ -99,13 +84,7 @@
         </inertial>
     </xacro:macro>
-    <!-- ########################## -->
-    <!--  Include additional files  -->
-    <!-- ########################## -->
-    <!-- Gazebo file for extra Gazebo options and motion driver-->
+    <!-- Include gazebo file -->
     <xacro:include filename="$(find robofetz_gazebo)/models/simple_diff_drive_robot/simple_diff_drive_robot.gazebo" />
-    <!-- ########################## -->
-    <!--  Define links and joints   -->
-    <!-- ########################## -->
-    <!-- Fictious link of the robot - we need to have this link otherwise Gazebo will complain -->
+    <!-- Links and joints -->
     <link name="$(arg prefix)base_footprint"> </link>
     <joint name="$(arg prefix)body_link_joint" type="fixed">
@@ -113,26 +92,20 @@
         <child link="$(arg prefix)body_link"/>
     </joint>
-    <!-- Body link of the robot -->
     <link name="$(arg prefix)body_link">
         <visual>
-            <geometry>
-                <box size="${a} ${c} ${b}" />
-            </geometry>
-            <!-- Displacement and orientation of the geometric center of the link with respec to the parent link -->
+            <geometry><box size="${a} ${c} ${b}" /></geometry>
             <origin rpy="0 0 0" xyz="0 0 ${s1}"/>
-        </visual>
-        <collision>
-            <geometry>
-                <box size="${a} ${c} ${b}" />
-            </geometry>
+            <material name="White"><color rgba="1 1 1 1"/></material>
+        </visual>
+        <collision>
+            <geometry><box size="${a} ${c} ${b}" /></geometry>
             <origin rpy="0 0 0" xyz="0 0 ${s1}"/>
         </collision>
         <xacro:inertia_body/>
     </link>
-    <!-- Top AprilTag link (added on top of the robot) -->
+    <!-- Top AprilTag -->
     <joint name="$(arg prefix)top_tag_joint" type="fixed">
         <parent link="$(arg prefix)body_link"/>
         <child link="$(arg prefix)top_apriltag_link"/>
-        <!-- Position the tag on top center of robot body, slightly offset to front -->
         <origin xyz="0 0 ${s1 + b/2 + tag_thickness/2}" rpy="0 0 0"/>
     </joint>
@@ -140,27 +113,17 @@
         <visual>
             <origin rpy="0 0 0" xyz="0 0 0"/>
-            <geometry>
-                <box size="${tag_size} ${tag_size} ${tag_thickness}"/>
-            </geometry>
-            <!-- Basic URDF material (fallback) -->
-            <material name="White">
-                <color rgba="1.0 1.0 1.0 1.0"/>
-            </material>
-        </visual>
-        <collision>
-            <origin rpy="0 0 0" xyz="0 0 0"/>
-            <geometry>
-                <box size="${tag_size} ${tag_size} ${tag_thickness}"/>
-            </geometry>
+            <geometry><box size="${tag_size} ${tag_size} ${tag_thickness}"/></geometry>
+            <material name="White"><color rgba="1 1 1 1"/></material>
+        </visual>
+        <collision>
+            <origin rpy="0 0 0" xyz="0 0 0"/>
+            <geometry><box size="${tag_size} ${tag_size} ${tag_thickness}"/></geometry>
         </collision>
         <xacro:inertia_tag/>
     </link>
-    <!-- Bottom AprilTag link (added on bottom of the robot) -->
+    <!-- Bottom AprilTag -->
     <joint name="$(arg prefix)bottom_tag_joint" type="fixed">
         <parent link="$(arg prefix)body_link"/>
         <child link="$(arg prefix)bottom_apriltag_link"/>
-        <!-- Position the tag on bottom center of robot body -->
-        <!-- Rotation 180 degrees around X axis to face downward -->
-        <!-- Position: s1 - b/2 - tag_thickness/2 (below the body) -->
         <origin xyz="0 0 ${s1 - b/2 - tag_thickness/2}" rpy="${pi_const} 0 0"/>
     </joint>
@@ -168,36 +131,22 @@
         <visual>
             <origin rpy="0 0 0" xyz="0 0 0"/>
-            <geometry>
-                <box size="${tag_size} ${tag_size} ${tag_thickness}"/>
-            </geometry>
-            <!-- Basic URDF material (fallback) -->
-            <material name="White">
-                <color rgba="1.0 1.0 1.0 1.0"/>
-            </material>
-        </visual>
-        <collision>
-            <origin rpy="0 0 0" xyz="0 0 0"/>
-            <geometry>
-                <box size="${tag_size} ${tag_size} ${tag_thickness}"/>
-            </geometry>
+            <geometry><box size="${tag_size} ${tag_size} ${tag_thickness}"/></geometry>
+            <material name="White"><color rgba="1 1 1 1"/></material>
+        </visual>
+        <collision>
+            <origin rpy="0 0 0" xyz="0 0 0"/>
+            <geometry><box size="${tag_size} ${tag_size} ${tag_thickness}"/></geometry>
         </collision>
         <xacro:inertia_tag/>
     </link>
-    <!-- Gazebo extension for Top AprilTag with PBR material -->
+    <!-- Gazebo PBR for top AprilTag -->
     <gazebo reference="$(arg prefix)top_apriltag_link">
-        <!-- Physics properties -->
         <kp>1000000.0</kp>
         <kd>100.0</kd>
         <mu1>0.5</mu1>
         <mu2>0.5</mu2>
-        <!-- Material override for Gazebo -->
         <material>Gazebo/White</material>
-        <!-- Visual override with PBR material -->
         <visual name="$(arg prefix)top_apriltag_visual">
-            <geometry>
-                <box>
-                    <size>${tag_size} ${tag_size} ${tag_thickness}</size>
-                </box>
-            </geometry>
+            <geometry><box><size>${tag_size} ${tag_size} ${tag_thickness}</size></box></geometry>
             <material>
                 <ambient>1 1 1 1</ambient>
@@ -214,20 +163,13 @@
         </visual>
     </gazebo>
-    <!-- Gazebo extension for Bottom AprilTag with PBR material -->
+    <!-- Gazebo PBR for bottom AprilTag -->
     <gazebo reference="$(arg prefix)bottom_apriltag_link">
-        <!-- Physics properties -->
         <kp>1000000.0</kp>
         <kd>100.0</kd>
         <mu1>0.5</mu1>
         <mu2>0.5</mu2>
-        <!-- Material override for Gazebo -->
         <material>Gazebo/White</material>
-        <!-- Visual override with PBR material -->
         <visual name="$(arg prefix)bottom_apriltag_visual">
-            <geometry>
-                <box>
-                    <size>${tag_size} ${tag_size} ${tag_thickness}</size>
-                </box>
-            </geometry>
+            <geometry><box><size>${tag_size} ${tag_size} ${tag_thickness}</size></box></geometry>
             <material>
                 <ambient>1 1 1 1</ambient>
@@ -236,5 +178,4 @@
                 <pbr>
                     <metal>
-                        <!-- Use a different texture for bottom tag if desired -->
                         <albedo_map>file://$(find robofetz_gazebo)/models/simple_diff_drive_robot/bottom_apriltag.png</albedo_map>
                         <roughness>0.5</roughness>
@@ -245,9 +186,9 @@
         </visual>
     </gazebo>
-    <!-- Wheel1 of the robot -->
-    <joint name="$(arg prefix)wheel1_joint" type="continuous" >
+    <!-- Wheels -->
+    <joint name="$(arg prefix)wheel1_joint" type="continuous">
         <parent link="$(arg prefix)body_link"/>
         <child link="$(arg prefix)wheel1_link"/>
-        <origin xyz="${-s2} ${-s4} ${r}" rpy="0 0 0" />
+        <origin xyz="${-s2} ${-s4} ${r}" rpy="0 0 0"/>
         <axis xyz="0 1 0"/>
         <limit effort="50000" velocity="10"/>
@@ -257,21 +198,17 @@
         <visual>
             <origin rpy="${pi_const/2} 0 0" xyz="0 0 0"/>
-            <geometry>
-                <cylinder length="${d}" radius="${r}"/>
-            </geometry>
-        </visual>
-        <collision>
-            <origin rpy="${pi_const/2} 0 0" xyz="0 0 0"/>
-            <geometry>
-                <cylinder length="${d}" radius="${r}"/>
-            </geometry>
+            <geometry><cylinder length="${d}" radius="${r}"/></geometry>
+            <material name="White"><color rgba="1 1 1 1"/></material>
+        </visual>
+        <collision>
+            <origin rpy="${pi_const/2} 0 0" xyz="0 0 0"/>
+            <geometry><cylinder length="${d}" radius="${r}"/></geometry>
         </collision>
         <xacro:inertia_wheel/>
     </link>
-    <!-- Wheel2 of the robot -->
-    <joint name="$(arg prefix)wheel2_joint" type="continuous" >
+    <joint name="$(arg prefix)wheel2_joint" type="continuous">
         <parent link="$(arg prefix)body_link"/>
         <child link="$(arg prefix)wheel2_link"/>
-        <origin xyz="${-s2} ${s4} ${r}" rpy="0 0 0" />
+        <origin xyz="${-s2} ${s4} ${r}" rpy="0 0 0"/>
         <axis xyz="0 1 0"/>
         <limit effort="50000" velocity="10"/>
@@ -281,36 +218,71 @@
         <visual>
             <origin rpy="${pi_const/2} 0 0" xyz="0 0 0"/>
-            <geometry>
-                <cylinder length="${d}" radius="${r}"/>
-            </geometry>
-        </visual>
-        <collision>
-            <origin rpy="${pi_const/2} 0 0" xyz="0 0 0"/>
-            <geometry>
-                <cylinder length="${d}" radius="${r}"/>
-            </geometry>
+            <geometry><cylinder length="${d}" radius="${r}"/></geometry>
+            <material name="White"><color rgba="1 1 1 1"/></material>
+        </visual>
+        <collision>
+            <origin rpy="${pi_const/2} 0 0" xyz="0 0 0"/>
+            <geometry><cylinder length="${d}" radius="${r}"/></geometry>
         </collision>
         <xacro:inertia_wheel/>
     </link>
-    <!-- Caster wheel of the robot -->
-    <joint name="$(arg prefix)caster_joint" type="fixed" >
-        <parent link="$(arg prefix)body_link"/>
-        <child link="$(arg prefix)caster_link"/>
-        <origin xyz="${s3} 0 ${r}" rpy="0 0 0" />
-    </joint>
-    <link name="$(arg prefix)caster_link">
-        <visual>
-            <origin rpy="0 0 0" xyz="0 0 0"/>
-            <geometry>
-                <sphere radius="${r}"/>
-            </geometry>
-        </visual>
-        <collision>
-            <origin rpy="0 0 0" xyz="0 0 0"/>
-            <geometry>
-                <sphere radius="${r}"/>
-            </geometry>
-        </collision>
-        <xacro:inertia_caster/>
-    </link>
+    <!-- Two upright boxes with top/bottom casters -->
+    <xacro:macro name="upright_with_casters" params="name y_offset">
+        <!-- Upright box -->
+        <joint name="$(arg prefix)${name}_joint" type="fixed">
+            <parent link="$(arg prefix)body_link"/>
+            <child link="$(arg prefix)${name}_link"/>
+            <origin xyz="${a/2+f} ${y_offset} ${r}" rpy="0 0 0"/>
+        </joint>
+        <link name="$(arg prefix)${name}_link">
+            <visual>
+                <origin rpy="0 0 0"/>
+                <geometry><box size="${support_width} ${support_width} ${support_height}"/></geometry>
+                <material name="White"><color rgba="1 1 1 1"/></material>
+            </visual>
+            <collision>
+                <origin rpy="0 0 0"/>
+                <geometry><box size="${support_width} ${support_width} ${support_height}"/></geometry>
+            </collision>
+            <xacro:inertia_support/>
+        </link>
+        <!-- Top caster -->
+        <joint name="$(arg prefix)${name}_top_caster_joint" type="fixed">
+            <parent link="$(arg prefix)${name}_link"/>
+            <child link="$(arg prefix)${name}_top_caster_link"/>
+            <origin xyz="0 0 ${support_height/2}" rpy="0 0 0"/>
+        </joint>
+        <link name="$(arg prefix)${name}_top_caster_link">
+            <visual>
+                <origin rpy="0 0 0"/>
+                <geometry><sphere radius="${f}"/></geometry>
+                <material name="White"><color rgba="1 1 1 1"/></material>
+            </visual>
+            <collision>
+                <origin rpy="0 0 0"/>
+                <geometry><sphere radius="${f}"/></geometry>
+            </collision>
+            <xacro:inertia_support/>
+        </link>
+        <!-- Bottom caster -->
+        <joint name="$(arg prefix)${name}_bottom_caster_joint" type="fixed">
+            <parent link="$(arg prefix)${name}_link"/>
+            <child link="$(arg prefix)${name}_bottom_caster_link"/>
+            <origin xyz="0 0 ${-support_height/2}" rpy="0 0 0"/>
+        </joint>
+        <link name="$(arg prefix)${name}_bottom_caster_link">
+            <visual>
+                <origin rpy="0 0 0"/>
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