Commit message: fixed prefix error

File: src/robofetz_gazebo/models/simple_diff_drive_opponent/simple_diff_drive_opponent.xacro (robot description, xacro)
@@ -4,4 +4,5 @@
     <!--   Geometry and constants   -->
     <!-- ########################## -->
+    <xacro:arg name="prefix" default="" />
     <!-- Pi -->
     <xacro:property name="pi_const" value="3.14159265" />
@@ -82,11 +83,11 @@
     <!-- ########################## -->
     <!-- Fictious link of the robot - we need to have this link otherwise Gazebo will complain -->
-    <link name="base_footprint"> </link>
-    <joint name="body_link_joint" type="fixed">
-        <parent link="base_footprint"/>
-        <child link="body_link"/>
+    <link name="$(arg prefix)base_footprint"> </link>
+    <joint name="$(arg prefix)body_link_joint" type="fixed">
+        <parent link="$(arg prefix)base_footprint"/>
+        <child link="$(arg prefix)body_link"/>
     </joint>
     <!-- Body link of the robot -->
-    <link name="body_link">
+    <link name="$(arg prefix)body_link">
         <visual>
             <geometry>
@@ -105,7 +106,7 @@
     </link>
     <!-- Wheel1 of the robot -->
-    <joint name="wheel1_joint" type="continuous" >
-        <parent link="body_link"/>
-        <child link="wheel1_link"/>
+    <joint name="$(arg prefix)wheel1_joint" type="continuous" >
+        <parent link="$(arg prefix)body_link"/>
+        <child link="$(arg prefix)wheel1_link"/>
         <origin xyz="${-s2} ${-s4} ${r}" rpy="0 0 0" />
         <axis xyz="0 1 0"/>
@@ -113,5 +114,5 @@
         <dynamics damping="1.0" friction="1.0"/>
     </joint>
-    <link name="wheel1_link">
+    <link name="$(arg prefix)wheel1_link">
         <visual>
             <origin rpy="${pi_const/2} 0 0" xyz="0 0 0"/>
@@ -129,7 +130,7 @@
     </link>
     <!-- Wheel2 of the robot -->
-    <joint name="wheel2_joint" type="continuous" >
-        <parent link="body_link"/>
-        <child link="wheel2_link"/>
+    <joint name="$(arg prefix)wheel2_joint" type="continuous" >
+        <parent link="$(arg prefix)body_link"/>
+        <child link="$(arg prefix)wheel2_link"/>
         <origin xyz="${-s2} ${s4} ${r}" rpy="0 0 0" />
         <axis xyz="0 1 0"/>
@@ -137,5 +138,5 @@
         <dynamics damping="1.0" friction="1.0"/>
     </joint>
-    <link name="wheel2_link">
+    <link name="$(arg prefix)wheel2_link">
         <visual>
             <origin rpy="${pi_const/2} 0 0" xyz="0 0 0"/>
@@ -153,10 +154,10 @@
     </link>
     <!-- Caster wheel of the robot -->
-    <joint name="caster_joint" type="fixed" >
-        <parent link="body_link"/>
-        <child link="caster_link"/>
+    <joint name="$(arg prefix)caster_joint" type="fixed" >
+        <parent link="$(arg prefix)body_link"/>
+        <child link="$(arg prefix)caster_link"/>
         <origin xyz="${s3} 0 ${r}" rpy="0 0 0" />
     </joint>
-    <link name="caster_link">
+    <link name="$(arg prefix)caster_link">
         <visual>
             <origin rpy="0 0 0" xyz="0 0 0"/>

File: src/robofetz_gazebo/models/simple_diff_drive_robot/simple_diff_drive_robot.xacro (robot description, xacro)
@@ -4,4 +4,5 @@
     <!--   Geometry and constants   -->
     <!-- ########################## -->
+    <xacro:arg name="prefix" default="" />
     <!-- Pi -->
     <xacro:property name="pi_const" value="3.14159265" />
@@ -82,11 +83,11 @@
     <!-- ########################## -->
     <!-- Fictious link of the robot - we need to have this link otherwise Gazebo will complain -->
-    <link name="base_footprint"> </link>
-    <joint name="body_link_joint" type="fixed">
-        <parent link="base_footprint"/>
-        <child link="body_link"/>
+    <link name="$(arg prefix)base_footprint"> </link>
+    <joint name="$(arg prefix)body_link_joint" type="fixed">
+        <parent link="$(arg prefix)base_footprint"/>
+        <child link="$(arg prefix)body_link"/>
     </joint>
     <!-- Body link of the robot -->
-    <link name="body_link">
+    <link name="$(arg prefix)body_link">
         <visual>
             <geometry>
@@ -105,7 +106,7 @@
     </link>
     <!-- Wheel1 of the robot -->
-    <joint name="wheel1_joint" type="continuous" >
-        <parent link="body_link"/>
-        <child link="wheel1_link"/>
+    <joint name="$(arg prefix)wheel1_joint" type="continuous" >
+        <parent link="$(arg prefix)body_link"/>
+        <child link="$(arg prefix)wheel1_link"/>
         <origin xyz="${-s2} ${-s4} ${r}" rpy="0 0 0" />
         <axis xyz="0 1 0"/>
@@ -113,5 +114,5 @@
         <dynamics damping="1.0" friction="1.0"/>
     </joint>
-    <link name="wheel1_link">
+    <link name="$(arg prefix)wheel1_link">
         <visual>
             <origin rpy="${pi_const/2} 0 0" xyz="0 0 0"/>
@@ -129,7 +130,7 @@
     </link>
     <!-- Wheel2 of the robot -->
-    <joint name="wheel2_joint" type="continuous" >
-        <parent link="body_link"/>
-        <child link="wheel2_link"/>
+    <joint name="$(arg prefix)wheel2_joint" type="continuous" >
+        <parent link="$(arg prefix)body_link"/>
+        <child link="$(arg prefix)wheel2_link"/>
         <origin xyz="${-s2} ${s4} ${r}" rpy="0 0 0" />
         <axis xyz="0 1 0"/>
@@ -137,5 +138,5 @@
         <dynamics damping="1.0" friction="1.0"/>
     </joint>
-    <link name="wheel2_link">
+    <link name="$(arg prefix)wheel2_link">
         <visual>
             <origin rpy="${pi_const/2} 0 0" xyz="0 0 0"/>
@@ -153,10 +154,10 @@
     </link>
     <!-- Caster wheel of the robot -->
-    <joint name="caster_joint" type="fixed" >
-        <parent link="body_link"/>
-        <child link="caster_link"/>
+    <joint name="$(arg prefix)caster_joint" type="fixed" >
+        <parent link="$(arg prefix)body_link"/>
+        <child link="$(arg prefix)caster_link"/>
         <origin xyz="${s3} 0 ${r}" rpy="0 0 0" />
     </joint>
-    <link name="caster_link">
+    <link name="$(arg prefix)caster_link">
         <visual>
             <origin rpy="0 0 0" xyz="0 0 0"/>

Commit message: cleanup of arg prefix

File: src/robofetz_gazebo/models/simple_diff_drive_opponent/simple_diff_drive_opponent.xacro (robot description, xacro)
@@ -4,5 +4,4 @@
     <!--   Geometry and constants   -->
     <!-- ########################## -->
-    <xacro:arg name="prefix" default="" />
     <!-- Pi -->
     <xacro:property name="pi_const" value="3.14159265" />
@@ -83,11 +82,11 @@
     <!-- ########################## -->
     <!-- Fictious link of the robot - we need to have this link otherwise Gazebo will complain -->
-    <link name="$(arg prefix)base_footprint"> </link>
-    <joint name="$(arg prefix)body_link_joint" type="fixed">
-        <parent link="$(arg prefix)base_footprint"/>
-        <child link="$(arg prefix)body_link"/>
+    <link name="base_footprint"> </link>
+    <joint name="body_link_joint" type="fixed">
+        <parent link="base_footprint"/>
+        <child link="body_link"/>
     </joint>
     <!-- Body link of the robot -->
-    <link name="$(arg prefix)body_link">
+    <link name="body_link">
         <visual>
             <geometry>
@@ -106,7 +105,7 @@
     </link>
     <!-- Wheel1 of the robot -->
-    <joint name="$(arg prefix)wheel1_joint" type="continuous" >
-        <parent link="$(arg prefix)body_link"/>
-        <child link="$(arg prefix)wheel1_link"/>
+    <joint name="wheel1_joint" type="continuous" >
+        <parent link="body_link"/>
+        <child link="wheel1_link"/>
         <origin xyz="${-s2} ${-s4} ${r}" rpy="0 0 0" />
         <axis xyz="0 1 0"/>
@@ -114,5 +113,5 @@
         <dynamics damping="1.0" friction="1.0"/>
     </joint>
-    <link name="$(arg prefix)wheel1_link">
+    <link name="wheel1_link">
         <visual>
             <origin rpy="${pi_const/2} 0 0" xyz="0 0 0"/>
@@ -130,7 +129,7 @@
     </link>
     <!-- Wheel2 of the robot -->
-    <joint name="$(arg prefix)wheel2_joint" type="continuous" >
-        <parent link="$(arg prefix)body_link"/>
-        <child link="$(arg prefix)wheel2_link"/>
+    <joint name="wheel2_joint" type="continuous" >
+        <parent link="body_link"/>
+        <child link="wheel2_link"/>
         <origin xyz="${-s2} ${s4} ${r}" rpy="0 0 0" />
         <axis xyz="0 1 0"/>
@@ -138,5 +137,5 @@
         <dynamics damping="1.0" friction="1.0"/>
     </joint>
-    <link name="$(arg prefix)wheel2_link">
+    <link name="wheel2_link">
         <visual>
             <origin rpy="${pi_const/2} 0 0" xyz="0 0 0"/>
@@ -154,10 +153,10 @@
     </link>
     <!-- Caster wheel of the robot -->
-    <joint name="$(arg prefix)caster_joint" type="fixed" >
-        <parent link="$(arg prefix)body_link"/>
-        <child link="$(arg prefix)caster_link"/>
+    <joint name="caster_joint" type="fixed" >
+        <parent link="body_link"/>
+        <child link="caster_link"/>
         <origin xyz="${s3} 0 ${r}" rpy="0 0 0" />
     </joint>
-    <link name="$(arg prefix)caster_link">
+    <link name="caster_link">
         <visual>
             <origin rpy="0 0 0" xyz="0 0 0"/>
