Commit message: it worksss

File: src/robot_description/urdf/robot.urdf.xacro (robot description, xacro)
@@ -122,4 +122,11 @@
         <xacro:inertia_tag/>
     </link>
+    <!-- Top AprilTag Optical Frame -->
+    <joint name="$(arg prefix)top_tag_optical_joint" type="fixed">
+        <parent link="$(arg prefix)top_apriltag_link"/>
+        <child link="$(arg prefix)top_apriltag_optical"/>
+        <origin xyz="0 0 0" rpy="0 ${pi_const} ${pi_const/2}"/>
+    </joint>
+    <link name="$(arg prefix)top_apriltag_optical"/>
     <!-- Bottom AprilTag -->
     <joint name="$(arg prefix)bottom_tag_joint" type="fixed">
@@ -140,4 +147,11 @@
         <xacro:inertia_tag/>
     </link>
+    <!-- Bottom AprilTag Optical Frame -->
+    <joint name="$(arg prefix)bottom_tag_optical_joint" type="fixed">
+        <parent link="$(arg prefix)bottom_apriltag_link"/>
+        <child link="$(arg prefix)bottom_apriltag_optical"/>
+                <origin xyz="0 0 0" rpy="0 0 ${pi_const/2}"/>
+    </joint>
+    <link name="$(arg prefix)bottom_apriltag_optical"/>
     <!-- Wheels -->
     <joint name="$(arg prefix)wheel1_joint" type="continuous">

Commit message: first efforts

File: src/robot_description/urdf/robot.urdf.xacro (robot description, xacro)
@@ -7,18 +7,25 @@
     <xacro:property name="pi_const" value="3.14159265" />
     <!-- Body Dimensions -->
-    <xacro:property name="a" value="0.140" />
-    <xacro:property name="b" value="0.054" />
-    <xacro:property name="c" value="0.14" />
+    <xacro:property name="a" value="0.0969" />
+    <xacro:property name="b" value="0.065" />
+    <xacro:property name="c" value="0.147" />
+    <xacro:property name="baseframe_offset_y" value="-0.02575" />
     <!-- Wheel and caster radius -->
-    <xacro:property name="r" value="0.034" />
+    <xacro:property name="r" value="0.0355" />
     <!-- Wheel width -->
-    <xacro:property name="d" value="0.026" />
+    <xacro:property name="d" value="0.01" />
     <!-- Wheel Offset to chassis in Y axis -->
-    <xacro:property name="wheel_offset_y" value="0.007" />
+    <xacro:property name="wheel_offset_x" value="-0.00925" />
+    <xacro:property name="wheel_offset_y" value="0.01" />
+    <!-- AprilTag properties -->
+    <xacro:property name="tag_size" value="0.094" />
+    <xacro:property name="tag_thickness" value="0.001" />
+    <xacro:property name="tag_mass" value="0.01" />
+    <xacro:property name="tag_offset_y" value="0.0" />
     <xacro:property name="s1" value="${r}" />
-    <xacro:property name="s2" value="${a/2.0-0.04075}" />
-    <xacro:property name="s3" value="${a+r}" />
-    <xacro:property name="s4" value="${c/2.0+d/2+wheel_offset_y}" />
+    <xacro:property name="s2" value="${a/2.0+wheel_offset_x}" />
+    <xacro:property name="s4" value="${c/2.0+wheel_offset_y}" />
     <!-- Upright support box dimensions (replacing cylinder) -->
+    <xacro:property name="weaponhold_length" value="51.5" />
     <xacro:property name="f" value="0.0049"/>
     <xacro:property name="support_width" value="${2*f}" />
@@ -46,8 +53,4 @@
     <xacro:property name="I_support_y" value="${(1.0/12.0)*m3*(support_width*support_width + support_height*support_height)}" />
     <xacro:property name="I_support_z" value="${(1.0/12.0)*m3*(support_width*support_width + support_width*support_width)}" />
-    <!-- AprilTag properties -->
-    <xacro:property name="tag_size" value="0.14" />
-    <xacro:property name="tag_thickness" value="0.001" />
-    <xacro:property name="tag_mass" value="0.01" />
     <!-- Complete inertia macros -->
     <xacro:macro name="inertia_body">
@@ -90,4 +93,5 @@
         <parent link="base_footprint"/>
         <child link="body_link"/>
+        <origin xyz="${baseframe_offset_y} 0 0" rpy="0 0 0"/>
     </joint>
     <link name="body_link">
@@ -107,5 +111,5 @@
         <parent link="body_link"/>
         <child link="top_apriltag_link"/>
-        <origin xyz="0 0 ${s1 + b/2 + tag_thickness/2}" rpy="0 0 0"/>
+        <origin xyz="${tag_offset_y} 0 ${s1 + b/2 + tag_thickness/2}" rpy="0 0 0"/>
     </joint>
     <link name="top_apriltag_link">
@@ -132,5 +136,5 @@
         <parent link="body_link"/>
         <child link="bottom_apriltag_link"/>
-        <origin xyz="0 0 ${s1 - b/2 - tag_thickness/2}" rpy="${pi_const} 0 0"/>
+        <origin xyz="${tag_offset_y} 0 ${s1 - b/2 - tag_thickness/2}" rpy="${pi_const} 0 0"/>
     </joint>
     <link name="bottom_apriltag_link">
@@ -157,5 +161,5 @@
         <parent link="body_link"/>
         <child link="right_wheel_link"/>
-        <origin xyz="${-s2} ${-s4} ${r}" rpy="0 0 0"/>
+        <origin xyz="${s2} ${-s4} ${r}" rpy="0 0 0"/>
         <axis xyz="0 1 0"/>
         <limit effort="50000" velocity="10"/>
@@ -177,5 +181,5 @@
         <parent link="body_link"/>
         <child link="left_wheel_link"/>
-        <origin xyz="${-s2} ${s4} ${r}" rpy="0 0 0"/>
+        <origin xyz="${s2} ${s4} ${r}" rpy="0 0 0"/>
         <axis xyz="0 1 0"/>
         <limit effort="50000" velocity="10"/>

Commit message: bot updated

File: src/robot_description/urdf/robot.urdf.xacro (robot description, xacro)
@@ -24,11 +24,14 @@
     <xacro:property name="tag_offset_y" value="0.0" />
     <xacro:property name="s1" value="${r}" />
-    <xacro:property name="s2" value="${a/2.0+wheel_offset_x}" />
+    <xacro:property name="s2" value="${wheel_offset_x}" />
     <xacro:property name="s4" value="${c/2.0+wheel_offset_y}" />
-    <!-- Upright support box dimensions (replacing cylinder) -->
-    <xacro:property name="weaponhold_length" value="51.5" />
-    <xacro:property name="f" value="0.0049"/>
-    <xacro:property name="support_width" value="${2*f}" />
-    <xacro:property name="support_height" value="${2*r-2*f}" />
+    <!-- Upright support box dimensions (independently definable) -->
+    <xacro:property name="support_width" value="0.0515" />      <!-- Width in X direction -->
+    <xacro:property name="support_depth" value="0.008" />     <!-- Depth in Y direction -->
+    <xacro:property name="support_height" value="0.065" />    <!-- Height in Z direction -->
+    <!-- Caster ball properties -->
+    <xacro:property name="caster_radius" value="${support_depth/2}" />    <!-- Radius of the ball casters -->
+    <xacro:property name="caster_mass" value="0.005" />      <!-- Mass of each caster ball -->
+    <xacro:property name="caster_offset" value="${support_height/2}" /> <!-- Position offset from box center -->
     <!-- ########################## -->
     <!--      Mass and inertia      -->
@@ -38,9 +41,10 @@
     <xacro:property name="d2" value="1430.0" />
     <xacro:property name="d3" value="1430.0" />
+    <xacro:property name="d4" value="1430.0" />  <!-- Density for caster balls -->
     <!-- Mass -->
     <xacro:property name="m1" value="${d1*a*b*c}" />
     <xacro:property name="m2" value="${d2*pi_const*r*r*d}" />
-    <!-- Updated mass calculation for box support -->
-    <xacro:property name="m3" value="${d3*support_width*support_width*support_height}" />
+    <xacro:property name="m3" value="${d3*support_width*support_depth*support_height}" />
+    <xacro:property name="m4" value="${d4 * (4.0/3.0) * pi_const * caster_radius * caster_radius * caster_radius}" /> <!-- Mass of caster ball -->
     <!-- Inertia -->
     <xacro:property name="Ix_body" value="${(1.0/12.0)*m1*(b*b+c*c)}" />
@@ -49,8 +53,10 @@
     <xacro:property name="Iz_wheel" value="${0.5*m2*r*r}" />
     <xacro:property name="I_wheel" value="${(1.0/12.0)*m2*(3.0*r*r+d*d)}" />
-    <!-- Updated inertia for box support -->
-    <xacro:property name="I_support_x" value="${(1.0/12.0)*m3*(support_width*support_width + support_height*support_height)}" />
+    <!-- Inertia for box support -->
+    <xacro:property name="I_support_x" value="${(1.0/12.0)*m3*(support_depth*support_depth + support_height*support_height)}" />
     <xacro:property name="I_support_y" value="${(1.0/12.0)*m3*(support_width*support_width + support_height*support_height)}" />
-    <xacro:property name="I_support_z" value="${(1.0/12.0)*m3*(support_width*support_width + support_width*support_width)}" />
+    <xacro:property name="I_support_z" value="${(1.0/12.0)*m3*(support_width*support_width + support_depth*support_depth)}" />
+    <!-- Inertia for caster ball (solid sphere) -->
+    <xacro:property name="I_caster" value="${(2.0/5.0)*m4*caster_radius*caster_radius}" />
     <!-- Complete inertia macros -->
     <xacro:macro name="inertia_body">
@@ -73,4 +79,11 @@
             <mass value="${m3}"/>
             <inertia ixx="${I_support_x}" ixy="0.0" ixz="0.0" iyy="${I_support_y}" iyz="0.0" izz="${I_support_z}" />
+        </inertial>
+    </xacro:macro>
+    <xacro:macro name="inertia_caster">
+        <inertial>
+            <origin rpy="0 0 0" xyz="0 0 0"/>
+            <mass value="${m4}"/>
+            <inertia ixx="${I_caster}" ixy="0.0" ixz="0.0" iyy="${I_caster}" iyz="0.0" izz="${I_caster}" />
         </inertial>
     </xacro:macro>
@@ -154,5 +167,5 @@
         <parent link="bottom_apriltag_link"/>
         <child link="bottom_apriltag_optical"/>
-                <origin xyz="0 0 0" rpy="0 0 ${pi_const/2}"/>
+        <origin xyz="0 0 0" rpy="0 0 ${pi_const/2}"/>
     </joint>
     <link name="bottom_apriltag_optical"/>
@@ -198,5 +211,5 @@
         <xacro:inertia_wheel/>
     </link>
-    <!-- Two upright boxes with top/bottom casters -->
+    <!-- Two upright boxes with independently definable top/bottom casters -->
     <xacro:macro name="upright_with_casters" params="name y_offset">
         <!-- Upright box -->
@@ -204,56 +217,56 @@
             <parent link="body_link"/>
             <child link="${name}_link"/>
-            <origin xyz="${a/2+f} ${y_offset} ${r}" rpy="0 0 0"/>
+            <origin xyz="${a/2 + support_width/2} ${y_offset} ${r}" rpy="0 0 0"/>
         </joint>
         <link name="${name}_link">
             <visual>
                 <origin rpy="0 0 0"/>
-                <geometry><box size="${support_width} ${support_width} ${support_height}"/></geometry>
+                <geometry><box size="${support_width} ${support_depth} ${support_height}"/></geometry>
                 <material name="White"><color rgba="1 1 1 1"/></material>
             </visual>
             <collision>
                 <origin rpy="0 0 0"/>
-                <geometry><box size="${support_width} ${support_width} ${support_height}"/></geometry>
+                <geometry><box size="${support_width} ${support_depth} ${support_height}"/></geometry>
             </collision>
             <xacro:inertia_support/>
         </link>
-        <!-- Top caster -->
+        <!-- Top caster ball -->
         <joint name="${name}_top_caster_joint" type="fixed">
             <parent link="${name}_link"/>
             <child link="${name}_top_caster_link"/>
-            <origin xyz="0 0 ${support_height/2}" rpy="0 0 0"/>
+            <origin xyz="${support_width/2-caster_radius} 0 ${caster_offset}" rpy="0 0 0"/>
         </joint>
         <link name="${name}_top_caster_link">
             <visual>
                 <origin rpy="0 0 0"/>
-                <geometry><sphere radius="${f}"/></geometry>
+                <geometry><sphere radius="${caster_radius}"/></geometry>
                 <material name="White"><color rgba="1 1 1 1"/></material>
             </visual>
             <collision>
                 <origin rpy="0 0 0"/>
-                <geometry><sphere radius="${f}"/></geometry>
+                <geometry><sphere radius="${caster_radius}"/></geometry>
             </collision>
-            <xacro:inertia_support/>
+            <xacro:inertia_caster/>
         </link>
-        <!-- Bottom caster -->
+        <!-- Bottom caster ball -->
         <joint name="${name}_bottom_caster_joint" type="fixed">
             <parent link="${name}_link"/>
             <child link="${name}_bottom_caster_link"/>
-            <origin xyz="0 0 ${-support_height/2}" rpy="0 0 0"/>
+            <origin xyz="${support_width/2-caster_radius} 0 ${-caster_offset}" rpy="0 0 0"/>
         </joint>
         <link name="${name}_bottom_caster_link">
             <visual>
                 <origin rpy="0 0 0"/>
-                <geometry><sphere radius="${f}"/></geometry>
+                <geometry><sphere radius="${caster_radius}"/></geometry>
                 <material name="White"><color rgba="1 1 1 1"/></material>
             </visual>
             <collision>
                 <origin rpy="0 0 0"/>
-                <geometry><sphere radius="${f}"/></geometry>
+                <geometry><sphere radius="${caster_radius}"/></geometry>
             </collision>
-            <xacro:inertia_support/>
+            <xacro:inertia_caster/>
         </link>
     </xacro:macro>
-    <xacro:upright_with_casters name="front_left_support" y_offset="${c/2 - f}"/>
-    <xacro:upright_with_casters name="front_right_support" y_offset="${-c/2 + f}"/>
+    <xacro:upright_with_casters name="front_left_support" y_offset="${c/2 - support_depth/2}"/>
+    <xacro:upright_with_casters name="front_right_support" y_offset="${-c/2 + support_depth/2}"/>
 </robot>
