Commit message: big reorga of robot description location

File: src/robot_description/urdf/gazebo/robot.gazebo.xacro (robot description, xacro)
@@ -51,4 +51,50 @@
         <material>Gazebo/Blue</material>
     </gazebo>
+    <!-- Gazebo PBR for top AprilTag -->
+    <gazebo reference="$(arg prefix)top_apriltag_link">
+        <kp>1000000.0</kp>
+        <kd>100.0</kd>
+        <mu1>0.5</mu1>
+        <mu2>0.5</mu2>
+        <material>Gazebo/White</material>
+        <visual name="$(arg prefix)top_apriltag_visual">
+            <geometry><box><size>${tag_size} ${tag_size} ${tag_thickness}</size></box></geometry>
+            <material>
+                <ambient>1 1 1 1</ambient>
+                <diffuse>1 1 1 1</diffuse>
+                <specular>0.5 0.5 0.5 1</specular>
+                <pbr>
+                    <metal>
+                        <albedo_map>file://$(find robot_description)/textures/top_apriltag.png</albedo_map>
+                        <roughness>0.5</roughness>
+                        <metalness>0.0</metalness>
+                    </metal>
+                </pbr>
+            </material>
+        </visual>
+    </gazebo>
+    <!-- Gazebo PBR for bottom AprilTag -->
+    <gazebo reference="$(arg prefix)bottom_apriltag_link">
+        <kp>1000000.0</kp>
+        <kd>100.0</kd>
+        <mu1>0.5</mu1>
+        <mu2>0.5</mu2>
+        <material>Gazebo/White</material>
+        <visual name="$(arg prefix)bottom_apriltag_visual">
+            <geometry><box><size>${tag_size} ${tag_size} ${tag_thickness}</size></box></geometry>
+            <material>
+                <ambient>1 1 1 1</ambient>
+                <diffuse>1 1 1 1</diffuse>
+                <specular>0.5 0.5 0.5 1</specular>
+                <pbr>
+                    <metal>
+                        <albedo_map>file://$(find robot_description)/textures/bottom_apriltag.png</albedo_map>
+                        <roughness>0.5</roughness>
+                        <metalness>0.0</metalness>
+                    </metal>
+                </pbr>
+            </material>
+        </visual>
+    </gazebo>
     <!-- Gazebo controller for differential drive robot -->
     <!-- controller plugin changed from gazebo classic to gazebo harmonic -->

File: src/robot_description/urdf/robot.urdf.xacro (robot description, xacro)
@@ -16,9 +16,9 @@
     <xacro:property name="d" value="0.026" />
     <!-- Wheel Offset to chassis in Y axis -->
-    <xacro:property name="e" value="0.00675" />
+    <xacro:property name="wheel_offset_y" value="0.007" />
     <xacro:property name="s1" value="${r}" />
     <xacro:property name="s2" value="${a/2.0-0.04075}" />
     <xacro:property name="s3" value="${a+r}" />
-    <xacro:property name="s4" value="${c/2.0+d/2+e}" />
+    <xacro:property name="s4" value="${c/2.0+d/2+wheel_offset_y}" />
     <!-- Upright support box dimensions (replacing cylinder) -->
     <xacro:property name="f" value="0.0049"/>
@@ -85,5 +85,5 @@
     </xacro:macro>
     <!-- Include gazebo file -->
-    <xacro:include filename="$(find robofetz_gazebo)/models/simple_diff_drive_robot/simple_diff_drive_robot.gazebo" />
+    <xacro:include filename="$(find robot_description)/urdf/gazebo/robot.gazebo.xacro" />
     <!-- Links and joints -->
     <link name="$(arg prefix)base_footprint"> </link>
@@ -140,50 +140,4 @@
         <xacro:inertia_tag/>
     </link>
-    <!-- Gazebo PBR for top AprilTag -->
-    <gazebo reference="$(arg prefix)top_apriltag_link">
-        <kp>1000000.0</kp>
-        <kd>100.0</kd>
-        <mu1>0.5</mu1>
-        <mu2>0.5</mu2>
-        <material>Gazebo/White</material>
-        <visual name="$(arg prefix)top_apriltag_visual">
-            <geometry><box><size>${tag_size} ${tag_size} ${tag_thickness}</size></box></geometry>
-            <material>
-                <ambient>1 1 1 1</ambient>
-                <diffuse>1 1 1 1</diffuse>
-                <specular>0.5 0.5 0.5 1</specular>
-                <pbr>
-                    <metal>
-                        <albedo_map>file://$(find robofetz_gazebo)/models/simple_diff_drive_robot/top_apriltag.png</albedo_map>
-                        <roughness>0.5</roughness>
-                        <metalness>0.0</metalness>
-                    </metal>
-                </pbr>
-            </material>
-        </visual>
-    </gazebo>
-    <!-- Gazebo PBR for bottom AprilTag -->
-    <gazebo reference="$(arg prefix)bottom_apriltag_link">
-        <kp>1000000.0</kp>
-        <kd>100.0</kd>
-        <mu1>0.5</mu1>
-        <mu2>0.5</mu2>
-        <material>Gazebo/White</material>
-        <visual name="$(arg prefix)bottom_apriltag_visual">
-            <geometry><box><size>${tag_size} ${tag_size} ${tag_thickness}</size></box></geometry>
-            <material>
-                <ambient>1 1 1 1</ambient>
-                <diffuse>1 1 1 1</diffuse>
-                <specular>0.5 0.5 0.5 1</specular>
-                <pbr>
-                    <metal>
-                        <albedo_map>file://$(find robofetz_gazebo)/models/simple_diff_drive_robot/bottom_apriltag.png</albedo_map>
-                        <roughness>0.5</roughness>
-                        <metalness>0.0</metalness>
-                    </metal>
-                </pbr>
-            </material>
-        </visual>
-    </gazebo>
     <!-- Wheels -->
     <joint name="$(arg prefix)wheel1_joint" type="continuous">

Commit message: fixed simulation time usage

File: src/robot_description/urdf/gazebo/robot.gazebo.xacro (robot description, xacro)
@@ -6,45 +6,45 @@
     <!-- match reference names with link names in robot.xacro ! -->
     <!-- wheel torques and speeds need now to be adjusted in robot.xacro with limit_effort and velocity under each joint-->
-    <gazebo reference="$(arg prefix)body_link">
+    <gazebo reference="body_link">
         <mu1>0.2</mu1>
         <mu2>0.2</mu2>
         <material>Gazebo/Green</material>
     </gazebo>
-    <gazebo reference="$(arg prefix)front_left_support_link">
+    <gazebo reference="front_left_support_link">
         <mu1>0.2</mu1>
         <mu2>0.2</mu2>
         <material>Gazebo/Green</material>
     </gazebo>
-    <gazebo reference="$(arg prefix)front_right_support_link">
+    <gazebo reference="front_right_support_link">
         <mu1>0.2</mu1>
         <mu2>0.2</mu2>
         <material>Gazebo/Green</material>
     </gazebo>
-    <gazebo reference="$(arg prefix)wheel1_link">
+    <gazebo reference="right_wheel_link">
         <mu1>0.8</mu1>
         <mu2>0.8</mu2>
         <material>Gazebo/Blue</material>
     </gazebo>
-    <gazebo reference="$(arg prefix)wheel2_link">
+    <gazebo reference="left_wheel_link">
         <mu1>0.8</mu1>
         <mu2>0.8</mu2>
         <material>Gazebo/Blue</material>
     </gazebo>
-    <gazebo reference="$(arg prefix)front_left_support_bottom_caster_link">
+    <gazebo reference="front_left_support_bottom_caster_link">
         <mu1>0.01</mu1>
         <mu2>0.01</mu2>
         <material>Gazebo/Blue</material>
     </gazebo>
-    <gazebo reference="$(arg prefix)front_left_support_top_caster_link">
+    <gazebo reference="front_left_support_top_caster_link">
         <mu1>0.01</mu1>
         <mu2>0.01</mu2>
         <material>Gazebo/Blue</material>
     </gazebo>
-     <gazebo reference="$(arg prefix)front_right_support_bottom_caster_link">
+     <gazebo reference="front_right_support_bottom_caster_link">
         <mu1>0.01</mu1>
         <mu2>0.01</mu2>
         <material>Gazebo/Blue</material>
     </gazebo>
-    <gazebo reference="$(arg prefix)front_right_support_top_caster_link">
+    <gazebo reference="front_right_support_top_caster_link">
         <mu1>0.01</mu1>
         <mu2>0.01</mu2>
@@ -52,5 +52,5 @@
     </gazebo>
     <!-- Gazebo PBR for top AprilTag -->
-    <gazebo reference="$(arg prefix)top_apriltag_link">
+    <gazebo reference="top_apriltag_link">
         <kp>1000000.0</kp>
         <kd>100.0</kd>
@@ -58,5 +58,5 @@
         <mu2>0.5</mu2>
         <material>Gazebo/White</material>
-        <visual name="$(arg prefix)top_apriltag_visual">
+        <visual name="top_apriltag_visual">
             <geometry><box><size>${tag_size} ${tag_size} ${tag_thickness}</size></box></geometry>
             <material>
@@ -75,5 +75,5 @@
     </gazebo>
     <!-- Gazebo PBR for bottom AprilTag -->
-    <gazebo reference="$(arg prefix)bottom_apriltag_link">
+    <gazebo reference="bottom_apriltag_link">
         <kp>1000000.0</kp>
         <kd>100.0</kd>
@@ -81,5 +81,5 @@
         <mu2>0.5</mu2>
         <material>Gazebo/White</material>
-        <visual name="$(arg prefix)bottom_apriltag_visual">
+        <visual name="bottom_apriltag_visual">
             <geometry><box><size>${tag_size} ${tag_size} ${tag_thickness}</size></box></geometry>
             <material>
@@ -104,6 +104,6 @@
         <plugin filename="gz-sim-diff-drive-system" name="gz::sim::systems::DiffDrive">
             <!-- wheels -->
-            <right_joint>$(arg prefix)wheel1_joint</right_joint>
-            <left_joint>$(arg prefix)wheel2_joint</left_joint>
+            <right_joint>right_wheel_joint</right_joint>
+            <left_joint>left_wheel_joint</left_joint>
             <!-- kinematics -->
             <wheel_separation>${2*s4}</wheel_separation>
@@ -124,6 +124,6 @@
           name="gz::sim::systems::JointStatePublisher">
             <topic>joint_states</topic>
-            <joint_name>wheel1_joint</joint_name>   <!-- arg prefix makes no difference here also / does not work see joint state echo -->
-            <joint_name>$(arg prefix)wheel2_joint</joint_name>
+            <joint_name>right_wheel_joint</joint_name>
+            <joint_name>left_wheel_joint</joint_name>
         </plugin>
         <!-- Publishes ground truth just for debugging. This is now done by arena_peception. -->

File: src/robot_description/urdf/robot.urdf.xacro (robot description, xacro)
@@ -4,5 +4,4 @@
     <!--   Geometry and constants   -->
     <!-- ########################## -->
-    <xacro:arg name="prefix" default="" />
     <!-- Pi -->
     <xacro:property name="pi_const" value="3.14159265" />
@@ -87,10 +86,10 @@
     <xacro:include filename="$(find robot_description)/urdf/gazebo/robot.gazebo.xacro" />
     <!-- Links and joints -->
-    <link name="$(arg prefix)base_footprint"> </link>
-    <joint name="$(arg prefix)body_link_joint" type="fixed">
-        <parent link="$(arg prefix)base_footprint"/>
-        <child link="$(arg prefix)body_link"/>
-    </joint>
-    <link name="$(arg prefix)body_link">
+    <link name="base_footprint"> </link>
+    <joint name="body_link_joint" type="fixed">
+        <parent link="base_footprint"/>
+        <child link="body_link"/>
+    </joint>
+    <link name="body_link">
         <visual>
             <geometry><box size="${a} ${c} ${b}" /></geometry>
@@ -105,10 +104,10 @@
     </link>
     <!-- Top AprilTag -->
-    <joint name="$(arg prefix)top_tag_joint" type="fixed">
-        <parent link="$(arg prefix)body_link"/>
-        <child link="$(arg prefix)top_apriltag_link"/>
+    <joint name="top_tag_joint" type="fixed">
+        <parent link="body_link"/>
+        <child link="top_apriltag_link"/>
         <origin xyz="0 0 ${s1 + b/2 + tag_thickness/2}" rpy="0 0 0"/>
     </joint>
-    <link name="$(arg prefix)top_apriltag_link">
+    <link name="top_apriltag_link">
         <visual>
             <origin rpy="0 0 0" xyz="0 0 0"/>
@@ -123,17 +122,17 @@
     </link>
     <!-- Top AprilTag Optical Frame -->
-    <joint name="$(arg prefix)top_tag_optical_joint" type="fixed">
-        <parent link="$(arg prefix)top_apriltag_link"/>
-        <child link="$(arg prefix)top_apriltag_optical"/>
+    <joint name="top_tag_optical_joint" type="fixed">
+        <parent link="top_apriltag_link"/>
+        <child link="top_apriltag_optical"/>
         <origin xyz="0 0 0" rpy="0 ${pi_const} ${pi_const/2}"/>
     </joint>
-    <link name="$(arg prefix)top_apriltag_optical"/>
+    <link name="top_apriltag_optical"/>
     <!-- Bottom AprilTag -->
-    <joint name="$(arg prefix)bottom_tag_joint" type="fixed">
-        <parent link="$(arg prefix)body_link"/>
-        <child link="$(arg prefix)bottom_apriltag_link"/>
+    <joint name="bottom_tag_joint" type="fixed">
+        <parent link="body_link"/>
+        <child link="bottom_apriltag_link"/>
         <origin xyz="0 0 ${s1 - b/2 - tag_thickness/2}" rpy="${pi_const} 0 0"/>
     </joint>
-    <link name="$(arg prefix)bottom_apriltag_link">
+    <link name="bottom_apriltag_link">
         <visual>
             <origin rpy="0 0 0" xyz="0 0 0"/>
@@ -148,14 +147,14 @@
     </link>
     <!-- Bottom AprilTag Optical Frame -->
-    <joint name="$(arg prefix)bottom_tag_optical_joint" type="fixed">
-        <parent link="$(arg prefix)bottom_apriltag_link"/>
-        <child link="$(arg prefix)bottom_apriltag_optical"/>
+    <joint name="bottom_tag_optical_joint" type="fixed">
+        <parent link="bottom_apriltag_link"/>
+        <child link="bottom_apriltag_optical"/>
                 <origin xyz="0 0 0" rpy="0 0 ${pi_const/2}"/>
     </joint>
-    <link name="$(arg prefix)bottom_apriltag_optical"/>
+    <link name="bottom_apriltag_optical"/>
     <!-- Wheels -->
-    <joint name="$(arg prefix)wheel1_joint" type="continuous">
-        <parent link="$(arg prefix)body_link"/>
-        <child link="$(arg prefix)wheel1_link"/>
+    <joint name="right_wheel_joint" type="continuous">
+        <parent link="body_link"/>
+        <child link="right_wheel_link"/>
         <origin xyz="${-s2} ${-s4} ${r}" rpy="0 0 0"/>
         <axis xyz="0 1 0"/>
@@ -163,5 +162,5 @@
         <dynamics damping="1.0" friction="1.0"/>
     </joint>
-    <link name="$(arg prefix)wheel1_link">
+    <link name="right_wheel_link">
         <visual>
             <origin rpy="${pi_const/2} 0 0" xyz="0 0 0"/>
@@ -175,7 +174,7 @@
         <xacro:inertia_wheel/>
     </link>
-    <joint name="$(arg prefix)wheel2_joint" type="continuous">
-        <parent link="$(arg prefix)body_link"/>
-        <child link="$(arg prefix)wheel2_link"/>
+    <joint name="left_wheel_joint" type="continuous">
+        <parent link="body_link"/>
+        <child link="left_wheel_link"/>
         <origin xyz="${-s2} ${s4} ${r}" rpy="0 0 0"/>
         <axis xyz="0 1 0"/>
@@ -183,5 +182,5 @@
         <dynamics damping="1.0" friction="1.0"/>
     </joint>
-    <link name="$(arg prefix)wheel2_link">
+    <link name="left_wheel_link">
         <visual>
             <origin rpy="${pi_const/2} 0 0" xyz="0 0 0"/>
@@ -198,10 +197,10 @@
     <xacro:macro name="upright_with_casters" params="name y_offset">
         <!-- Upright box -->
-        <joint name="$(arg prefix)${name}_joint" type="fixed">
-            <parent link="$(arg prefix)body_link"/>
-            <child link="$(arg prefix)${name}_link"/>
+        <joint name="${name}_joint" type="fixed">
+            <parent link="body_link"/>
+            <child link="${name}_link"/>
             <origin xyz="${a/2+f} ${y_offset} ${r}" rpy="0 0 0"/>
         </joint>
-        <link name="$(arg prefix)${name}_link">
+        <link name="${name}_link">
             <visual>
                 <origin rpy="0 0 0"/>
@@ -216,10 +215,10 @@
         </link>
         <!-- Top caster -->
-        <joint name="$(arg prefix)${name}_top_caster_joint" type="fixed">
-            <parent link="$(arg prefix)${name}_link"/>
-            <child link="$(arg prefix)${name}_top_caster_link"/>
+        <joint name="${name}_top_caster_joint" type="fixed">
+            <parent link="${name}_link"/>
+            <child link="${name}_top_caster_link"/>
             <origin xyz="0 0 ${support_height/2}" rpy="0 0 0"/>
         </joint>
-        <link name="$(arg prefix)${name}_top_caster_link">
+        <link name="${name}_top_caster_link">
             <visual>
                 <origin rpy="0 0 0"/>
@@ -234,10 +233,10 @@
         </link>
         <!-- Bottom caster -->
-        <joint name="$(arg prefix)${name}_bottom_caster_joint" type="fixed">
-            <parent link="$(arg prefix)${name}_link"/>
-            <child link="$(arg prefix)${name}_bottom_caster_link"/>
+        <joint name="${name}_bottom_caster_joint" type="fixed">
+            <parent link="${name}_link"/>
+            <child link="${name}_bottom_caster_link"/>
             <origin xyz="0 0 ${-support_height/2}" rpy="0 0 0"/>
         </joint>
-        <link name="$(arg prefix)${name}_bottom_caster_link">
+        <link name="${name}_bottom_caster_link">
             <visual>
                 <origin rpy="0 0 0"/>

Commit message: weapon added

File: src/robot_description/urdf/gazebo/robot.gazebo.xacro (robot description, xacro)
@@ -50,4 +50,9 @@
         <mu2>0.01</mu2>
         <material>Gazebo/Blue</material>
+    </gazebo>
+    <gazebo reference="weapon_link">
+        <mu1>0.01</mu1>
+        <mu2>0.01</mu2>
+        <material>Gazebo/Grey</material>
     </gazebo>
     <!-- Gazebo PBR for top AprilTag -->

File: src/robot_description/urdf/robot.urdf.xacro (robot description, xacro)
@@ -23,4 +23,11 @@
     <xacro:property name="tag_mass" value="0.01" />
     <xacro:property name="tag_offset_y" value="0.0" />
+    <!-- Weapon properties -->
+    <xacro:property name="weapon_length" value="0.060" />
+    <xacro:property name="weapon_width" value="0.124" />
+    <xacro:property name="weapon_height" value="0.010" />
+    <xacro:property name="weapon_offset_x" value="0.08495" />
+    <xacro:property name="weapon_mass" value="0.1" />       <!-- Mass of weapon (kg) -->
+    <xacro:property name="weapon_density" value="1430.0" /> <!-- Material density -->
     <xacro:property name="s1" value="${r}" />
     <xacro:property name="s2" value="${wheel_offset_x}" />
@@ -42,4 +49,5 @@
     <xacro:property name="d3" value="1430.0" />
     <xacro:property name="d4" value="1430.0" />  <!-- Density for caster balls -->
+    <xacro:property name="d5" value="${weapon_density}" /> <!-- Density for weapon -->
     <!-- Mass -->
     <xacro:property name="m1" value="${d1*a*b*c}" />
@@ -47,4 +55,5 @@
     <xacro:property name="m3" value="${d3*support_width*support_depth*support_height}" />
     <xacro:property name="m4" value="${d4 * (4.0/3.0) * pi_const * caster_radius * caster_radius * caster_radius}" /> <!-- Mass of caster ball -->
+    <xacro:property name="m5" value="${d5*weapon_length*weapon_width*weapon_height}" /> <!-- Mass of weapon -->
     <!-- Inertia -->
     <xacro:property name="Ix_body" value="${(1.0/12.0)*m1*(b*b+c*c)}" />
@@ -59,4 +68,8 @@
     <!-- Inertia for caster ball (solid sphere) -->
     <xacro:property name="I_caster" value="${(2.0/5.0)*m4*caster_radius*caster_radius}" />
+    <!-- Inertia for weapon (rectangular box) -->
+    <xacro:property name="Ix_weapon" value="${(1.0/12.0)*m5*(weapon_width*weapon_width + weapon_height*weapon_height)}" />
+    <xacro:property name="Iy_weapon" value="${(1.0/12.0)*m5*(weapon_length*weapon_length + weapon_height*weapon_height)}" />
+    <xacro:property name="Iz_weapon" value="${(1.0/12.0)*m5*(weapon_length*weapon_length + weapon_width*weapon_width)}" />
     <!-- Complete inertia macros -->
     <xacro:macro name="inertia_body">
@@ -86,4 +99,11 @@
             <mass value="${m4}"/>
             <inertia ixx="${I_caster}" ixy="0.0" ixz="0.0" iyy="${I_caster}" iyz="0.0" izz="${I_caster}" />
+        </inertial>
+    </xacro:macro>
+    <xacro:macro name="inertia_weapon">
+        <inertial>
+            <origin rpy="0 0 0" xyz="0 0 0"/>
+            <mass value="${m5}"/>
+            <inertia ixx="${Ix_weapon}" ixy="0.0" ixz="0.0" iyy="${Iy_weapon}" iyz="0.0" izz="${Iz_weapon}" />
         </inertial>
     </xacro:macro>
@@ -119,4 +139,22 @@
         </collision>
         <xacro:inertia_body/>
+    </link>
+    <!-- Weapon Link -->
+    <joint name="weapon_joint" type="fixed">
+        <parent link="body_link"/>
+        <child link="weapon_link"/>
+        <origin xyz="${weapon_offset_x} 0 ${s1}" rpy="0 0 0"/>
+    </joint>
+    <link name="weapon_link">
+        <visual>
+            <origin rpy="0 0 0" xyz="0 0 0"/>
+            <geometry><box size="${weapon_length} ${weapon_width} ${weapon_height}"/></geometry>
+            <material name="Red"><color rgba="1 0 0 1"/></material>
+        </visual>
+        <collision>
+            <origin rpy="0 0 0" xyz="0 0 0"/>
+            <geometry><box size="${weapon_length} ${weapon_width} ${weapon_height}"/></geometry>
+        </collision>
+        <xacro:inertia_weapon/>
     </link>
     <!-- Top AprilTag -->
